File: mfs/shiield/final_shield/1.brd (EAGLE design)
At the start: 53.3 x 101.6 mm, 31 parts, among them IC1 L298

Commit message: pcb files updated
Routing:
- net GND: track 0.00 -> 271.7 mm
- net 5V: track 0.00 -> 165.5 mm
- net VIN: track 0.00 -> 90.9 mm
- net 28: track 0.00 -> 73.1 mm
- net 26: track 0.00 -> 69.4 mm
- net R2: track 0.00 -> 65.8 mm, vias 0 -> 1
- net 4: track 0.00 -> 65.1 mm, vias 0 -> 1
- net 3V3: track 0.00 -> 64.2 mm, vias 0 -> 1
- net N$3: track 0.00 -> 63.7 mm
- net T2: track 0.00 -> 55.5 mm, vias 0 -> 2
- net 2: track 0.00 -> 55.3 mm
- net 24: track 0.00 -> 53.8 mm, vias 0 -> 1
- net 22: track 0.00 -> 51.4 mm
- net R1: track 0.00 -> 50.0 mm
- net N$4: track 0.00 -> 47.1 mm
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